Commit message: fixed urdf, wrote PIP instead of DIP

File: ros2/telekinesis/robot_hand/robot_pybullet.urdf (robot description, URDF)
Before this commit: robot NEW_HAND_7_14, 20 links, 19 joints
Links:
- link Index_DIP: geometry collision mesh filename=Index_DIP.STL; visual mesh filename=Index_DIP.STL
